Commit message: Add igris_moveit_config and update source files
Adds both_arms group with waist in SRDF, self collision test node,
collision avoidance planner, and updates to igris driver, teleop, and URDF.

Co-Authored-By: Claude Opus 4.6 (1M context) <noreply@anthropic.com>

File: src/urdf_igris/urdf/igris_c_v2.urdf (robot description, URDF)
Before this commit: robot IGRIS_C, 34 links, 33 joints
Links:
- link Left_Hand: geometry collision box size=0.15 0.05 0.2; visual mesh filename=file:///home/josh/Igris_c_ros2_ws/src/urdf_igris/urdf/meshe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 scale=0.01 0.01 0.01
- link Link_Ankle_Pitch_Left: geometry collision mesh filename=file:///home/josh/Igris_c_ros2_ws/src/urdf_igris/urdf/meshe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 scale=0.01 0.01 0.01; visual mesh filename=file:///home/josh/Igris_c_ros2_ws/src/urdf_igris/urdf/meshe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 scale=0.01 0.01 0.01
- link Link_Ankle_Pitch_Right: geometry collision mesh filename=file:///home/josh/Igris_c_ros2_ws/src/urdf_igris/urdf/meshe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 scale=0.01 0.01 0.01; visual mesh filename=file:///home/josh/Igris_c_ros2_ws/src/urdf_igris/urdf/meshe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 scale=0.01 0.01 0.01
- link Link_Ankle_Roll_Left: geometry collision box size=0.2 0.07 0.014; visual mesh filename=file:///home/josh/Igris_c_ros2_ws/src/urdf_igris/urdf/meshe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 scale=0.01 0.01 0.01
- link Link_Ankle_Roll_Right: geometry collision box size=0.2 0.07 0.014; visual mesh filename=file:///home/josh/Igris_c_ros2_ws/src/urdf_igris/urdf/meshe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 scale=0.01 0.01 0.01
- link Link_Elbow_Pitch_Left: geometry collision mesh filename=file:///home/josh/Igris_c_ros2_ws/src/urdf_igris/urdf/meshe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 scale=0.01 0.01 0.01; visual mesh filename=file:///home/josh/Igris_c_ros2_ws/src/urdf_igris/urdf/meshe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 scale=0.01 0.01 0.01
- link Link_Elbow_Pitch_Right: geometry collision mesh filename=file:///home/josh/Igris_c_ros2_ws/src/urdf_igris/urdf/meshe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 scale=0.01 0.01 0.01; visual mesh filename=file:///home/josh/Igris_c_ros2_ws/src/urdf_igris/urdf/meshe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 scale=0.01 0.01 0.01
- link Link_Hip_Pitch_Left: geometry collision mesh filename=file:///home/josh/Igris_c_ros2_ws/src/urdf_igris/urdf/meshe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 scale=0.01 0.01 0.01; visual mesh filename=file:///home/josh/Igris_c_ros2_ws/src/urdf_igris/urdf/meshe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 scale=0.01 0.01 0.01
- link Link_Hip_Pitch_Right: geometry collision mesh filename=file:///home/josh/Igris_c_ros2_ws/src/urdf_igris/urdf/meshe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 scale=0.01 0.01 0.01; visual mesh filename=file:///home/josh/Igris_c_ros2_ws/src/urdf_igris/urdf/meshe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 scale=0.01 0.01 0.01
- link Link_Hip_Roll_Left: geometry collision box size=0.16 0.12 0.12; visual mesh filename=file:///home/josh/Igris_c_ros2_ws/src/urdf_igris/urdf/meshe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 scale=0.01 0.01 0.01
- link Link_Hip_Roll_Right: geometry collision box size=0.16 0.12 0.12; visual mesh filename=file:///home/josh/Igris_c_ros2_ws/src/urdf_igris/urdf/meshe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 scale=0.01 0.01 0.01
- link Link_Hip_Yaw_Left: geometry collision mesh filename=file:///home/josh/Igris_c_ros2_ws/src/urdf_igris/urdf/meshe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 scale=0.01 0.01 0.01; visual mesh filename=file:///home/josh/Igris_c_ros2_ws/src/urdf_igris/urdf/meshe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 scale=0.01 0.01 0.01
- link Link_Hip_Yaw_Right: geometry collision mesh filename=file:///home/josh/Igris_c_ros2_ws/src/urdf_igris/urdf/meshe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 scale=0.01 0.01 0.01; visual mesh filename=file:///home/josh/Igris_c_ros2_ws/src/urdf_igris/urdf/meshe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 scale=0.01 0.01 0.01
- link Link_Knee_Pitch_Left: geometry collision box size=0.15 0.1 0.25; visual mesh filename=file:///home/josh/Igris_c_ros2_ws/src/urdf_igris/urdf/meshe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 scale=0.01 0.01 0.01
- link Link_Knee_Pitch_Right: geometry collision box size=0.15 0.1 0.25; visual mesh filename=file:///home/josh/Igris_c_ros2_ws/src/urdf_igris/urdf/meshe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 scale=0.01 0.01 0.01
- link Link_Neck_Pitch: geometry collision box size=0.2 0.15 0.18; visual mesh filename=file:///home/josh/Igris_c_ros2_ws/src/urdf_igris/urdf/meshe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 scale=0.01 0.01 0.01
- link Link_Neck_Yaw: geometry collision mesh filename=file:///home/josh/Igris_c_ros2_ws/src/urdf_igris/urdf/meshe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 scale=0.01 0.01 0.01; visual mesh filename=file:///home/josh/Igris_c_ros2_ws/src/urdf_igris/urdf/meshe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 scale=0.01 0.01 0.01
- link Link_Shoulder_Pitch_Left: geometry collision mesh filename=file:///home/josh/Igris_c_ros2_ws/src/urdf_igris/urdf/meshe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 scale=0.01 0.01 0.01; visual mesh filename=file:///home/josh/Igris_c_ros2_ws/src/urdf_igris/urdf/meshe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 scale=0.01 0.01 0.01
- link Link_Shoulder_Pitch_Right: geometry collision mesh filename=file:///home/josh/Igris_c_ros2_ws/src/urdf_igris/urdf/meshe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 scale=0.01 0.01 0.01; visual mesh filename=file:///home/josh/Igris_c_ros2_ws/src/urdf_igris/urdf/meshe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 scale=0.01 0.01 0.01
- link Link_Shoulder_Roll_Left: geometry collision mesh filename=file:///home/josh/Igris_c_ros2_ws/src/urdf_igris/urdf/meshe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 scale=0.01 0.01 0.01; visual mesh filename=file:///home/josh/Igris_c_ros2_ws/src/urdf_igris/urdf/meshe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 scale=0.01 0.01 0.01
- link Link_Shoulder_Roll_Right: geometry collision mesh filename=file:///home/josh/Igris_c_ros2_ws/src/urdf_igris/urdf/meshe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 scale=0.01 0.01 0.01; visual mesh filename=file:///home/josh/Igris_c_ros2_ws/src/urdf_igris/urdf/meshe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 scale=0.01 0.01 0.01
- link Link_Shoulder_Yaw_Left: geometry collision mesh filename=file:///home/josh/Igris_c_ros2_ws/src/urdf_igris/urdf/meshe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 scale=0.01 0.01 0.01; visual mesh filename=file:///home/josh/Igris_c_ros2_ws/src/urdf_igris/urdf/meshe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 scale=0.01 0.01 0.01
- link Link_Shoulder_Yaw_Right: geometry collision mesh filename=file:///home/josh/Igris_c_ros2_ws/src/urdf_igris/urdf/meshe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 scale=0.01 0.01 0.01; visual mesh filename=file:///home/josh/Igris_c_ros2_ws/src/urdf_igris/urdf/meshe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 scale=0.01 0.01 0.01
- link Link_Waist_Pitch: geometry collision mesh filename=file:///home/josh/Igris_c_ros2_ws/src/urdf_igris/urdf/meshe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 scale=0.01 0.01 0.01; visual mesh filename=file:///home/josh/Igris_c_ros2_ws/src/urdf_igris/urdf/meshe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 scale=0.01 0.01 0.01
- link Link_Waist_Roll: geometry collision mesh filename=file:///home/josh/Igris_c_ros2_ws/src/urdf_igris/urdf/meshe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 scale=0.01 0.01 0.01; visual mesh filename=file:///home/josh/Igris_c_ros2_ws/src/urdf_igris/urdf/meshe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 scale=0.01 0.01 0.01
- link Link_Waist_Yaw: geometry collision mesh filename=file:///home/josh/Igris_c_ros2_ws/src/urdf_igris/urdf/meshe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 scale=0.01 0.01 0.01; visual mesh filename=file:///home/josh/Igris_c_ros2_ws/src/urdf_igris/urdf/meshe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 scale=0.01 0.01 0.01
- link Link_Wrist_Pitch_Left: geometry collision mesh filename=file:///home/josh/Igris_c_ros2_ws/src/urdf_igris/urdf/meshe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 scale=0.01 0.01 0.01; visual mesh filename=file:///home/josh/Igris_c_ros2_ws/src/urdf_igris/urdf/meshe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 scale=0.01 0.01 0.01
- link Link_Wrist_Pitch_Right: geometry collision mesh filename=file:///home/josh/Igris_c_ros2_ws/src/urdf_igris/urdf/meshe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 scale=0.01 0.01 0.01; visual mesh filename=file:///home/josh/Igris_c_ros2_ws/src/urdf_igris/urdf/meshe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 scale=0.01 0.01 0.01
- link Link_Wrist_Roll_Left: geometry collision mesh filename=file:///home/josh/Igris_c_ros2_ws/src/urdf_igris/urdf/meshe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 scale=0.01 0.01 0.01; visual mesh filename=file:///home/josh/Igris_c_ros2_ws/src/urdf_igris/urdf/meshe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 scale=0.01 0.01 0.01
- link Link_Wrist_Roll_Right: geometry collision mesh filename=file:///home/josh/Igris_c_ros2_ws/src/urdf_igris/urdf/meshe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 scale=0.01 0.01 0.01; visual mesh filename=file:///home/josh/Igris_c_ros2_ws/src/urdf_igris/urdf/meshe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 scale=0.01 0.01 0.01
- link Link_Wrist_Yaw_Left: geometry collision cylinder length=0.24 radius=0.05; visual mesh filename=file:///home/josh/Igris_c_ros2_ws/src/urdf_igris/urdf/meshe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 scale=0.01 0.01 0.01
- link Link_Wrist_Yaw_Right: geometry collision cylinder length=0.24 radius=0.05; visual mesh filename=file:///home/josh/Igris_c_ros2_ws/src/urdf_igris/urdf/meshe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 scale=0.01 0.01 0.01
- link Right_Hand: geometry collision box size=0.15 0.05 0.2; visual mesh filename=file:///home/josh/Igris_c_ros2_ws/src/urdf_igris/urdf/meshe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 scale=0.01 0.01 0.01
- link base_link: geometry collision box size=0.22 0.23 0.33; visual mesh filename=file:///home/josh/Igris_c_ros2_ws/src/urdf_igris/urdf/meshe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 scale=0.01 0.01 0.01
Joints:
- joint 13_Joint_Ankle_Pitch_Right: limit lower=-0.698131701 upper=0.698131701 effort=1000 velocity=100.0 -> lower=-0.523598776 upper=0.523598776 effort=1000 velocity=100.0
- joint 14_Joint_Ankle_Roll_Right: limit lower=-0.261799388 upper=0.261799388 effort=1000 velocity=100.0 -> lower=-0.174532925 upper=0.174532925 effort=1000 velocity=100.0
- joint 20_Joint_Wrist_Roll_Left: limit lower=-1.221730476 upper=0.872664626 effort=1000 velocity=100.0 -> lower=-1.221730476 upper=1.221730476 effort=1000 velocity=100.0
- joint 21_Joint_Wrist_Pitch_Left: limit lower=-0.698131701 upper=0.698131701 effort=1000 velocity=100.0 -> lower=-1.698131701 upper=1.698131701 effort=1000 velocity=100.0
- joint 27_Joint_Wrist_Roll_Right: limit lower=-0.872664626 upper=1.221730476 effort=1000 velocity=100.0 -> lower=-1.221730476 upper=1.221730476 effort=1000 velocity=100.0
- joint 28_Joint_Wrist_Pitch_Right: limit lower=-0.698131701 upper=0.698131701 effort=1000 velocity=100.0 -> lower=-1.698131701 upper=1.698131701 effort=1000 velocity=100.0
